File: hardware/kicad/youverse-hardware.kicad_sch (KiCad schematic)
At the start: 12 parts, among them J1 USB_B_Micro, U1 ESP32-WROOM-32, U2 DHT11, U3 AMS1117-3.3

Commit message: add updated folders
Parts:
- removed C1, C2, C3: C, symbol Device:C
- removed U3: AMS1117-3.3, Package_TO_SOT_SMD:SOT-223-3_TabPin2, symbol Regulator_Linear:AMS1117-3.3
- added C5: 10 uF, Capacitor_THT:CP_Radial_D5.0mm_P2.00mm, symbol Device:C
- added J2: PIR sensor, Connector_PinHeader_2.54mm:PinHeader_1x03_P2.54mm_Vertical, symbol Connector_Generic:Conn_01x03
- added R6: Potentiometer, Potentiometer_THT:Potentiometer_Bourns_3296W_Vertical, symbol Simulation_SPICE:Potentiometer
- added U4: ER_OLEDM0.91_1x-I2C, Display:ER_OLEDM0.91_1x-I2C, symbol Display_Graphic:ER_OLEDM0.91_1x-I2C
- added U5: AP2112K-3.3, Package_TO_SOT_SMD:SOT-23-5, symbol Regulator_Linear:AP2112K-3.3
- C4: value C -> 10 uF; footprint (none) -> Capacitor_THT:CP_Radial_D5.0mm_P2.00mm
- J1: footprint (none) -> Connector_USB:USB_Micro-B_Molex-105017-0001
- R1: footprint (none) -> Resistor_THT:R_Axial_DIN0207_L6.3mm_D2.5mm_P10.16mm_Horizontal
- R2, R3: value R -> 10K; footprint (none) -> Resistor_THT:R_Axial_DIN0207_L6.3mm_D2.5mm_P10.16mm_Horizontal
- R4: value R -> 10k; footprint (none) -> Resistor_THT:R_Axial_DIN0207_L6.3mm_D2.5mm_P10.16mm_Horizontal
Connections:
- net +3V3: now also C5.2, J2.1 (Pin_1), R6.1, U4.1 (GND), U4.2 (VCC), U5.5 (VOUT)
- net GND: now also C5.1, J2.3 (Pin_3), R6.3, U5.2 (GND)
- net GPIO27_PIR: now reaches U1.12 (IO27)
- net GPIO27_PIR: now also J2.2 (Pin_2)
- net GPIO21_POT: now reaches U1.33 (IO21)
- net GPIO21_POT: now also U4.4 (SDA)
- net GPIO22_POT: now reaches U1.36 (IO22)
- net GPIO22_POT: now also U4.3 (SCL)
- net GPIO35_POT: now reaches U1.7 (IO35)
- net GPIO35_POT: now also R6.2
- net at C4.2, J1.1 (VBUS): now also U5.1 (VIN), U5.3 (EN)
Other:
- note added: "16-8-2026"
- moved on the sheet: C4, J1, R1, R2, R3, R4, U2
